Commit message: controller added

File: urdf/roboter_zusammenbau.urdf (robot description, URDF)
Before this commit: robot roboter_zusammenbau, 27 links, 26 joints
Links:
- removed link dummy
- added link world
- link Gripper_Rot_Plate: mass 0.110297257500002 -> 0.11029725831735
- link X_Axis: mass 3.40836171067752 -> 3.40836170630821
- link Y_Axis: mass 5.1487838864562 -> 5.14878388645621
- link Z_Axis: mass 2.9874598652384 -> 2.98745986427534
Joints:
- removed joint EQ_joint
- removed joint dummy_joint
- added joint EQ_Joint: type prismatic, parent Z_Axis, child EQ, origin xyz=0.2365 0.032258 -0.254 rpy=0 0 0, axis 0 0 1, limit lower=0 upper=0.02 effort=100 velocity=0.05
- added joint world_joint: type fixed, parent world, child base_link, origin xyz=0 0 0 rpy=0 0 0
- joint Camera_Calibartion_Joint: limit lower=0 upper=0.04 effort=100 velocity=0.05 -> lower=-0.04 upper=0.0 effort=100 velocity=0.05
- joint Gripper_Rot_Plate_Joint: limit lower=0 upper=628319 effort=100 velocity=0.05 -> lower=0 upper=3.14 effort=100 velocity=0.1; origin xyz=0.0075 0.09 -0.333 rpy=0 0 0 -> xyz=0.00750000000000184 0.0900000062570289 -0.389620000000001 rpy=0 0 0
- joint X_Axis_Joint: limit lower=0 upper=1 effort=100 velocity=0.05 -> lower=-0.745 upper=0.055 effort=100 velocity=0.05
- joint Y_Axis_Joint: limit lower=0 upper=0.5 effort=100 velocity=0.05 -> lower=-0.425 upper=0.2505 effort=100 velocity=0.05; origin xyz=0.41353 -0.39197 0.0625 rpy=0 0 0 -> xyz=0.1115 -0.39197 0.0625 rpy=0 0 0
- joint Z_Axis_Joint: axis 0 0 1 -> 0 0 -1; limit lower=0 upper=0.3 effort=100 velocity=0.05 -> lower=-0.05262 upper=0.045 effort=100 velocity=0.5; origin xyz=-0.001 0.46653 0.28252 rpy=0 0 0 -> xyz=-0.001 0.4962 0.28252 rpy=0 0 0

Commit message: Aktuallisiertes Robotermodell

File: urdf/roboter_zusammenbau.urdf (robot description, URDF)
Before this commit: robot roboter_zusammenbau, 27 links, 26 joints
Links:
- link Glue_Cartridge_Flap: mass 0.0179277924431148 -> 0.0179277924431147
- link Gonio_Left_Stage_1_Upper: mass 0.578798887684806 -> 0.578798857286943
- link Gonio_Left_Stage_2_Upper: mass 0.0270626709955924 -> 0.0270626702476323
- link Gonio_Right_Mount_Lower: mass 0.193859171974624 -> 0.193859196114997
- link Gonio_Right_Mount_Upper: mass 0.0762325940447469 -> 0.0762325967846099
Joints:
- joint EQ_Joint: limit lower=0 upper=0.02 effort=100 velocity=0.05 -> lower=-0.05109 upper=0 effort=100 velocity=0.05; origin xyz=0.2365 0.032258 -0.254 rpy=0 0 0 -> xyz=0.236500000000002 0.0322575758254203 -0.258000000000002 rpy=0 0 0
- joint Glue_Cartridge_Flap_Joint: origin xyz=0.16314 0.102 -0.4115 rpy=0 0 0 -> xyz=0.075000000000002 0.0545000062570288 -0.360000000000001 rpy=0 0 0
- joint Gonio_Base_Left_Joint: origin xyz=0.7525 0.6845 0.1 rpy=0 0 0 -> xyz=0.752500000000035 0.684500000000037 0.100000000000003 rpy=0 0 0
- joint Gonio_Left_Stage_1_Upper_Joint: origin xyz=0.1565 0.11 0.2125 rpy=0 0 0 -> xyz=0.156499999999957 0.109999999999947 0.212499999999997 rpy=0 0 0
- joint Gonio_Left_Stage_2_Upper_Joint: axis 0 -0.99592 0.09025 -> 0 -1 0; origin xyz=-0.04 0.024898 -0.0022563 rpy=0 0 0 -> xyz=-0.04 0.025 0 rpy=0 0 0
- joint Gonio_Right_Mount_Lower_joint: origin xyz=-0.025217 -0.051199 -0.010968 rpy=-0.090394 -0.021325 0.0019328 -> xyz=-0.0255632010662045 -0.05 -0.0149680967303876 rpy=0 0.00124847209372143 0
- joint Gonio_Right_Mount_Upper_Joint: origin xyz=0.00054449 0 0 rpy=0.090373 0.021412 0 -> xyz=0.000544493897539577 0 0 rpy=0 -0.00124847209372143 0
- joint Gonio_Right_Stage_1_Upper_joint: origin xyz=0.0125 0.0325 0.282 rpy=0 0 0 -> xyz=0.0125000000000001 0.0325000000000001 0.281999999999999 rpy=0 0 0
- joint Gonio_Right_Stage_2_Upper_Joint: origin xyz=0.0325 0.032498 0.00032062 rpy=0.0098655 0.0024365 2.4038E-05 -> xyz=0.0325 0.0324984184257152 0.000320624121260105 rpy=0.00986554689296988 0.00243647716593582 2.40379358152113E-05
- joint Gonio_base_Rigth_Joint: origin xyz=0.84378 0.7682 0.29928 rpy=-0.090394 -0.021325 0.0019328 -> xyz=0.843436798933783 0.769499999999991 0.297531903269611 rpy=0 0.00124847209373138 0
- joint Gripper_Rot_Plate_Joint: origin xyz=0.00750000000000184 0.0900000062570289 -0.389620000000001 rpy=0 0 0 -> xyz=0.00750000000000206 0.0900000062570289 -0.337000000000001 rpy=0 0 0
- joint Nest_Joint: origin xyz=-0.0325 -0.065 -0.05 rpy=0 0 0 -> xyz=-0.0324999999999999 -0.065 -0.0499999999999998 rpy=0 0 0
- joint Stage_1_Gonio_Right_Joint: origin xyz=-0.49265 0.018632 -0.17514 rpy=0.090373 0.021412 0 -> xyz=-0.488205660861556 0.00050000000005054 -0.185441558777103 rpy=0 -0.00124847209373138 0

Commit message: Cam1 als einzelnes Modell

File: urdf/roboter_zusammenbau.urdf (robot description, URDF)
Before this commit: robot roboter_zusammenbau, 27 links, 26 joints
Links:
- added link Camera_Module_Z_Axis, mass 0.0744906107551848; collision mesh filename=ppackage://roboter_zusammenbau/meshes/Camera_Module_Z_Axis.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; visual mesh filename=package://roboter_zusammenbau/meshes/Camera_Module_Z_Axis.S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
Joints:
- added joint Camera_Module_Z_Axis_Joint: type fixed, parent Z_Axis, child Camera_Module_Z_Axis, origin xyz=0.0795000000000031 0.0685000209707082 -0.181500000000001 rpy=0 0 0, axis 0 0 0
- joint Gonio_Left_Stage_1_Upper_Joint: limit lower=-0.78539816339745 upper=0.78539816339745 effort=100 velocity=0.01 -> lower=-0.78539816339745 upper=0.78539816339745 effort=100 velocity=0.1
- joint Gonio_Left_Stage_2_Upper_Joint: limit lower=-0.78539816339745 upper=0.78539816339745 effort=100 velocity=0.01 -> lower=-0.78539816339745 upper=0.78539816339745 effort=100 velocity=0.1
- joint Gonio_Right_Stage_1_Upper_joint: limit lower=-0.087266 upper=0.087266 effort=100 velocity=0.01 -> lower=-0.087266 upper=0.087266 effort=100 velocity=0.1
- joint Gonio_Right_Stage_2_Upper_Joint: limit lower=-0.17453 upper=0.17453 effort=100 velocity=0.01 -> lower=-0.17453 upper=0.17453 effort=100 velocity=0.1
- joint UV_Module_Left_Joint: limit lower=0 upper=0.05 effort=100 velocity=0.05 -> lower=-0.05 upper=0.0 effort=100 velocity=0.05
- joint UV_Module_Right_Joint: limit lower=0 upper=0.05 effort=100 velocity=0.05 -> lower=-0.05 upper=0.0 effort=100 velocity=0.05
