Commit message: implement controllers for XYZ axis

File: urdf/main.xacro (robot description, xacro)
@@ -4,3 +4,4 @@
   xmlns:xacro="https://ros.org/wiki/xacro">
     <xacro:include filename="$(find roboter_zusammenbau)/urdf/roboter_zusammenbau.urdf" />
+    <xacro:include filename="$(find roboter_zusammenbau)/urdf/controller.urdf" />
 </robot>

File: urdf/roboter_zusammenbau.urdf (robot description, URDF)
Before this commit: robot roboter_zusammenbau, 26 links, 25 joints
Links:
- added link dummy
Joints:
- added joint dummy_joint: type fixed, parent dummy, child base_link

Commit message: Projekt in pm_robot umbenannt

File: urdf/main.xacro (robot description, xacro)
@@ -1,7 +1,7 @@
 <?xml version="1.0" encoding="utf-8"?>
 <robot
-  name="roboter_zusammenbau"
+  name="pm_robot"
   xmlns:xacro="https://ros.org/wiki/xacro">
-    <xacro:include filename="$(find roboter_zusammenbau)/urdf/roboter_zusammenbau.urdf" />
-    <xacro:include filename="$(find roboter_zusammenbau)/urdf/controller.urdf" />
+    <xacro:include filename="$(find pm_robot)/urdf/pm_robot.urdf" />
+    <xacro:include filename="$(find pm_robot)/urdf/controller.urdf" />
 </robot>

File: urdf/pm_robot.urdf (robot description, URDF)
Before this commit: robot roboter_zusammenbau, 28 links, 27 joints
Links:
- link Camera_Calibration: geometry collision mesh filename=package://pm_robot/meshes/Camera_Calibration.STL; visual mesh filename=package://pm_robot/meshes/Camera_Calibration.STL
- link Camera_Module_Z_Axis: geometry collision mesh filename=ppackage://pm_robot/meshes/Camera_Module_Z_Axis.STL; visual mesh filename=package://pm_robot/meshes/Camera_Module_Z_Axis.STL
- link Camera_System: geometry collision mesh filename=package://pm_robot/meshes/Camera_System.STL; visual mesh filename=package://pm_robot/meshes/Camera_System.STL
- link EQ: geometry collision mesh filename=package://pm_robot/meshes/EQ.STL; visual mesh filename=package://pm_robot/meshes/EQ.STL
- link Glue_Cartridge: geometry collision mesh filename=package://pm_robot/meshes/Glue_Cartridge.STL; visual mesh filename=package://pm_robot/meshes/Glue_Cartridge.STL
- link Glue_Cartridge_Flap: geometry collision mesh filename=package://pm_robot/meshes/Glue_Cartridge_Flap.STL; visual mesh filename=package://pm_robot/meshes/Glue_Cartridge_Flap.STL
- link Gonio_Base_Left: geometry collision mesh filename=package://pm_robot/meshes/Gonio_Base_Left.STL; visual mesh filename=package://pm_robot/meshes/Gonio_Base_Left.STL
- link Gonio_Base_Rigth: geometry collision mesh filename=package://pm_robot/meshes/Gonio_Base_Rigth.STL; visual mesh filename=package://pm_robot/meshes/Gonio_Base_Rigth.STL
- link Gonio_Left_Stage_1_Upper: geometry collision mesh filename=package://pm_robot/meshes/Gonio_Left_Stage_1_Upper.STL; visual mesh filename=package://pm_robot/meshes/Gonio_Left_Stage_1_Upper.STL
- link Gonio_Left_Stage_2_Upper: geometry collision mesh filename=package://pm_robot/meshes/Gonio_Left_Stage_2_Upper.STL; visual mesh filename=package://pm_robot/meshes/Gonio_Left_Stage_2_Upper.STL
- link Gonio_Right_Mount_Lower: geometry collision mesh filename=package://pm_robot/meshes/Gonio_Right_Mount_Lower.STL; visual mesh filename=package://pm_robot/meshes/Gonio_Right_Mount_Lower.STL
- link Gonio_Right_Mount_Upper: geometry collision mesh filename=package://pm_robot/meshes/Gonio_Right_Mount_Upper.STL; visual mesh filename=package://pm_robot/meshes/Gonio_Right_Mount_Upper.STL
- link Gonio_Right_Stage_1_Upper: geometry collision mesh filename=package://pm_robot/meshes/Gonio_Right_Stage_1_Upper.STL; visual mesh filename=package://pm_robot/meshes/Gonio_Right_Stage_1_Upper.STL
- link Gonio_Right_Stage_2_Upper: geometry collision mesh filename=package://pm_robot/meshes/Gonio_Right_Stage_2_Upper.STL; visual mesh filename=package://pm_robot/meshes/Gonio_Right_Stage_2_Upper.STL
- link Gripper: geometry collision mesh filename=package://pm_robot/meshes/Gripper.STL; visual mesh filename=package://pm_robot/meshes/Gripper.STL
- link Gripper_Rot_Plate: geometry collision mesh filename=package://pm_robot/meshes/Gripper_Rot_Plate.STL; visual mesh filename=package://pm_robot/meshes/Gripper_Rot_Plate.STL
- link Nest: geometry collision mesh filename=package://pm_robot/meshes/Nest.STL; visual mesh filename=package://pm_robot/meshes/Nest.STL
- link Stage_1_Gonio_Right: geometry collision mesh filename=package://pm_robot/meshes/Stage_1_Gonio_Right.STL; visual mesh filename=package://pm_robot/meshes/Stage_1_Gonio_Right.STL
- link Test_Station: geometry collision mesh filename=package://pm_robot/meshes/Test_Station.STL; visual mesh filename=package://pm_robot/meshes/Test_Station.STL
- link UV_Cart_Left: geometry collision mesh filename=package://pm_robot/meshes/UV_Cart_Left.STL; visual mesh filename=package://pm_robot/meshes/UV_Cart_Left.STL
- link UV_Cart_Right: geometry collision mesh filename=package://pm_robot/meshes/UV_Cart_Right.STL; visual mesh filename=package://pm_robot/meshes/UV_Cart_Right.STL
- link UV_Module_Left: geometry collision mesh filename=package://pm_robot/meshes/UV_Module_Left.STL; visual mesh filename=package://pm_robot/meshes/UV_Module_Left.STL
- link UV_Module_Right: geometry collision mesh filename=package://pm_robot/meshes/UV_Module_Right.STL; visual mesh filename=package://pm_robot/meshes/UV_Module_Right.STL
- link X_Axis: geometry collision mesh filename=package://pm_robot/meshes/X_Axis.STL; visual mesh filename=package://pm_robot/meshes/X_Axis.STL
- link Y_Axis: geometry collision mesh filename=package://pm_robot/meshes/Y_Axis.STL; visual mesh filename=package://pm_robot/meshes/Y_Axis.STL
- link Z_Axis: geometry collision mesh filename=package://pm_robot/meshes/Z_Axis.STL; visual mesh filename=package://pm_robot/meshes/Z_Axis.STL
- link base_link: geometry collision mesh filename=package://pm_robot/meshes/base_link.STL; visual mesh filename=package://pm_robot/meshes/base_link.STL
