Commit message: Camera added to the model

File: urdf/pm_robot.urdf (robot description, URDF)
Before this commit: robot pm_robot, 28 links, 27 joints
Links:
- added link camera_link
- added link camera_link_optical
Joints:
- added joint camera_joint: type fixed, parent Camera_Module_Z_Axis, child camera_link, origin xyz=0.02 0.021 -0.16 rpy=0 ${pi/2} 0 
- added joint camera_optical_joint: type fixed, parent Camera_Module_Z_Axis, child camera_link_optical, origin xyz=0 0 0 rpy=${-pi/2} 0 ${-pi/2} 

Commit message: Abhishek 24.11

File: urdf/pm_robot.urdf (robot description, URDF)
Before this commit: robot pm_robot, 30 links, 29 joints
Links:
- link Camera_Module_Z_Axis: geometry collision mesh filename=package://pm_robot/meshes/Camera_Module_Z_Axis.STL; visual mesh filename=package://pm_robot/meshes/Camera_Module_Z_Axis.STL
Joints:
- joint Z_Axis_Joint: limit lower=-0.05262 upper=0.045 effort=100 velocity=0.5 -> lower=-0.05262 upper=0.8 effort=100 velocity=0.5
- joint camera_joint: origin xyz=0.02 0.021 -0.16 rpy=0 ${pi/2} 0  -> xyz=0.02 0.021 -0.16 rpy=0 1.570796 0 
- joint camera_optical_joint: origin xyz=0 0 0 rpy=${-pi/2} 0 ${-pi/2}  -> xyz=0 0 0 rpy=-1.570796 0 -1.570796 

Commit message: Z-Axis angepasst

File: urdf/pm_robot.urdf (robot description, URDF)
Before this commit: robot pm_robot, 30 links, 29 joints
Links:
- link Camera_Module_Z_Axis: mass 0.0744906107551848 -> 0.0744906107551854
- link Glue_Cartridge: mass 0.072567178977958 -> 0.0725671789065893
- link Glue_Cartridge_Flap: mass 0.0179277924431147 -> 0.0179277924431146
- link UV_Cart_Right: mass 0.127959263608561 -> 0.127959263593804
- link Z_Axis: mass 2.98745986427534 -> 2.90435657697672
Joints:
- joint Camera_Module_Z_Axis_Joint: origin xyz=0.0795000000000031 0.0685000209707082 -0.181500000000001 rpy=0 0 0 -> xyz=0.0795000000000243 0.068500020970708 -0.233999999999991 rpy=0 0 0
- joint EQ_Joint: limit lower=-0.05109 upper=0 effort=100 velocity=0.05 -> lower=0 upper=0.02 effort=100 velocity=0.05; origin xyz=0.236500000000002 0.0322575758254203 -0.258000000000002 rpy=0 0 0 -> xyz=0.236500000000024 0.0322575758254202 -0.310499999999992 rpy=0 0 0
- joint Glue_Cartridge_Flap_Joint: origin xyz=0.075000000000002 0.0545000062570288 -0.360000000000001 rpy=0 0 0 -> xyz=0.0750000000000233 0.0545000062570286 -0.412499999999991 rpy=0 0 0
- joint Glue_Cartridge_Joint: origin xyz=0.1715 0.0582 -0.2855 rpy=0 0 0 -> xyz=0.171500000000024 0.0582000062570286 -0.341999999999991 rpy=0 0 0
- joint Gripper_Joint: origin xyz=0 0 -0.0255 rpy=0 0 0 -> xyz=0 0 -0.0255000000000101 rpy=0 0 0
- joint Gripper_Rot_Plate_Joint: limit lower=0 upper=3.14 effort=100 velocity=0.1 -> lower=0 upper=628319 effort=100 velocity=0.05; origin xyz=0.00750000000000206 0.0900000062570289 -0.337000000000001 rpy=0 0 0 -> xyz=0.00750000000002338 0.0900000062570287 -0.389499999999991 rpy=0 0 0
- joint UV_Cart_Left_Joint: limit lower=0 upper=0.1 effort=100 velocity=0.05 -> lower=-0.05 upper=0.095 effort=100 velocity=0.05; origin xyz=0.0065 0.23118 0.2526 rpy=0 0 0 -> xyz=0.00649999999276624 0.231179999755626 0.252599999998818 rpy=0 0 0
- joint UV_Cart_Right_Joint: limit lower=0 upper=0.1 effort=0.05 velocity=100 -> lower=-0.045 upper=0.045 effort=0.05 velocity=100; origin xyz=0.0065 0.05118 0.2526 rpy=0 0 0 -> xyz=0.00649999999276935 0.0511799999883173 0.252599999998818 rpy=0 0 0
- joint UV_Module_Left_Joint: limit lower=-0.05 upper=0.0 effort=100 velocity=0.05 -> lower=0.045 upper=0.045 effort=100 velocity=0.05; origin xyz=0.092383 0.02382 0.0276 rpy=0 0 0 -> xyz=0.109999999999999 0.0238200000000034 0.0276000000000078 rpy=0 0 0
- joint UV_Module_Right_Joint: limit lower=-0.05 upper=0.0 effort=100 velocity=0.05 -> lower=0 upper=0.05 effort=100 velocity=0.05; origin xyz=0.11255 -0.08618 0.0276 rpy=0 0 0 -> xyz=0.109999999941829 -0.0861800000000014 0.0276000000000078 rpy=0 0 0
- joint Z_Axis_Joint: axis 0 0 -1 -> 0 0 1; limit lower=-0.05262 upper=0.8 effort=100 velocity=0.5 -> lower=-0.05262 upper=0.055 effort=100 velocity=0.05; origin xyz=-0.001 0.4962 0.28252 rpy=0 0 0 -> xyz=-0.000999999553101816 0.496199999543101 0.2825180193463 rpy=0 0 0
